File: detector/detector.sch (KiCad schematic (older format))
At the start: 48 parts, among them CON1 AVR-ISP-6, IC1 ATTINY441-SSU, P1 LASER, P2 BATTERY, P3 CONN_01X01, P4 CONN_01X01, P5 CONN_01X01, Q1 OPTO_NPN, Q2 OPTO_NPN, Q3 OPTO_NPN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

Commit message: Rename
Connections:
- net MATRIX_OUT: now also R3.1
- net THRESHOLD: no longer R3.1
Changed lines of the file:
@@
 LIBS:contrib
 LIBS:valves
-LIBS:receiver-cache
+LIBS:detector-cache
 LIBS:mysensors_radios
 EELAYER 25 0
@@
 encoding utf-8
 Sheet 1 1
-Title "Laser maze receiver"
+Title "Laser maze detector"
 Date "2016-03-25"
 Rev "1"
@@
 $EndComp
 $Comp
-L GND #PWR9
+L GND #PWR01
 U 1 1 56DA93BD
 P 3450 1800
-F 0 "#PWR9" H 3450 1550 50  0001 C CNN
+F 0 "#PWR01" H 3450 1550 50  0001 C CNN
 F 1 "GND" H 3458 1626 50  0000 C CNN
 F 2 "" H 3450 1800 60  0000 C CNN
@@
 $EndComp
 $Comp
-L VCC #PWR15
+L VCC #PWR02
 U 1 1 56DA951F
 P 4200 1500
-F 0 "#PWR15" H 4200 1350 50  0001 C CNN
+F 0 "#PWR02" H 4200 1350 50  0001 C CNN
 F 1 "VCC" H 4220 1674 50  0000 C CNN
 F 2 "" H 4200 1500 60  0000 C CNN
@@
 $EndComp
 $Comp
-L VAA #PWR5
+L VAA #PWR03
 U 1 1 56DA953F
 P 2150 1500
-F 0 "#PWR5" H 2150 1350 50  0001 C CNN
+F 0 "#PWR03" H 2150 1350 50  0001 C CNN
 F 1 "VAA" H 2170 1674 50  0000 C CNN
 F 2 "" H 2150 1500 60  0000 C CNN
@@
 $EndComp
 $Comp
-L VCC #PWR1
+L VCC #PWR04
 U 1 1 56DA95CF
 P 1050 2850
-F 0 "#PWR1" H 1050 2700 50  0001 C CNN
+F 0 "#PWR04" H 1050 2700 50  0001 C CNN
 F 1 "VCC" H 1070 3024 50  0000 C CNN
 F 2 "" H 1050 2850 60  0000 C CNN
@@
 $EndComp
 $Comp
-L GND #PWR2
+L GND #PWR05
 U 1 1 56DA9D61
 P 1050 4050
-F 0 "#PWR2" H 1050 3800 50  0001 C CNN
+F 0 "#PWR05" H 1050 3800 50  0001 C CNN
 F 1 "GND" H 1058 3876 50  0000 C CNN
 F 2 "" H 1050 4050 60  0000 C CNN
@@
 $EndComp
 $Comp
-L GND #PWR25
+L GND #PWR06
 U 1 1 56DA9DB4
 P 8600 3950
-F 0 "#PWR25" H 8600 3700 50  0001 C CNN
+F 0 "#PWR06" H 8600 3700 50  0001 C CNN
 F 1 "GND" H 8608 3776 50  0000 C CNN
 F 2 "" H 8600 3950 60  0000 C CNN
@@
 $EndComp
 $Comp
-L GND #PWR19
+L GND #PWR07
 U 1 1 56DAA419
 P 5850 1850
-F 0 "#PWR19" H 5850 1600 50  0001 C CNN
+F 0 "#PWR07" H 5850 1600 50  0001 C CNN
 F 1 "GND" H 5858 1676 50  0000 C CNN
 F 2 "" H 5850 1850 60  0000 C CNN
@@
 $EndComp
 $Comp
-L GND #PWR20
+L GND #PWR08
 U 1 1 56DAA463
 P 7150 1450
-F 0 "#PWR20" H 7150 1200 50  0001 C CNN
+F 0 "#PWR08" H 7150 1200 50  0001 C CNN
 F 1 "GND" H 7158 1276 50  0000 C CNN
 F 2 "" H 7150 1450 60  0000 C CNN
@@
 $EndComp
 $Comp
-L GND #PWR22
+L GND #PWR09
 U 1 1 56DAA4AE
 P 7400 2700
-F 0 "#PWR22" H 7400 2450 50  0001 C CNN
+F 0 "#PWR09" H 7400 2450 50  0001 C CNN
 F 1 "GND" H 7408 2526 50  0000 C CNN
 F 2 "" H 7400 2700 60  0000 C CNN
@@
 $EndComp
 $Comp
-L VCC #PWR24
+L VCC #PWR010
 U 1 1 56DAA83E
 P 8600 2600
-F 0 "#PWR24" H 8600 2450 50  0001 C CNN
+F 0 "#PWR010" H 8600 2450 50  0001 C CNN
 F 1 "VCC" H 8620 2774 50  0000 C CNN
 F 2 "" H 8600 2600 60  0000 C CNN
@@
 $EndComp
 $Comp
-L GND #PWR26
+L GND #PWR011
 U 1 1 56DABB35
 P 8650 5450
-F 0 "#PWR26" H 8650 5200 50  0001 C CNN
+F 0 "#PWR011" H 8650 5200 50  0001 C CNN
 F 1 "GND" H 8658 5276 50  0000 C CNN
 F 2 "" H 8650 5450 60  0000 C CNN
@@
 $EndComp
 $Comp
-L GND #PWR27
+L GND #PWR012
 U 1 1 56DABC05
 P 9650 3250
-F 0 "#PWR27" H 9650 3000 50  0001 C CNN
+F 0 "#PWR012" H 9650 3000 50  0001 C CNN
 F 1 "GND" H 9658 3076 50  0000 C CNN
 F 2 "" H 9650 3250 60  0000 C CNN
@@
 $EndComp
 $Comp
-L GND #PWR23
+L GND #PWR013
 U 1 1 56DABD6D
 P 8350 4750
-F 0 "#PWR23" H 8350 4500 50  0001 C CNN
+F 0 "#PWR013" H 8350 4500 50  0001 C CNN
 F 1 "GND" H 8358 4576 50  0000 C CNN
 F 2 "" H 8350 4750 60  0000 C CNN
@@
 $EndComp
 $Comp
-L GND #PWR28
+L GND #PWR014
 U 1 1 56DAC359
 P 9700 5250
-F 0 "#PWR28" H 9700 5000 50  0001 C CNN
+F 0 "#PWR014" H 9700 5000 50  0001 C CNN
 F 1 "GND" H 9708 5076 50  0000 C CNN
 F 2 "" H 9700 5250 60  0000 C CNN
@@
 $EndComp
 $Comp
-L VCC #PWR29
+L VCC #PWR015
 U 1 1 56DAC41F
 P 10550 4150
-F 0 "#PWR29" H 10550 4000 50  0001 C CNN
+F 0 "#PWR015" H 10550 4000 50  0001 C CNN
 F 1 "VCC" H 10570 4324 50  0000 C CNN
 F 2 "" H 10550 4150 60  0000 C CNN
@@
 $EndComp
 $Comp
-L GND #PWR18
+L GND #PWR016
 U 1 1 56DAFB30
 P 5750 4750
-F 0 "#PWR18" H 5750 4500 50  0001 C CNN
+F 0 "#PWR016" H 5750 4500 50  0001 C CNN
 F 1 "GND" H 5758 4576 50  0000 C CNN
 F 2 "" H 5750 4750 60  0000 C CNN
@@
 $EndComp
 $Comp
-L VCC #PWR17
+L VCC #PWR017
 U 1 1 56DAFBC7
 P 5750 4150
-F 0 "#PWR17" H 5750 4000 50  0001 C CNN
+F 0 "#PWR017" H 5750 4000 50  0001 C CNN
 F 1 "VCC" H 5770 4324 50  0000 C CNN
 F 2 "" H 5750 4150 60  0000 C CNN
@@
 $EndComp
 $Comp
-L GND #PWR16
+L GND #PWR018
 U 1 1 56DB26B9
 P 5500 7500
-F 0 "#PWR16" H 5500 7250 50  0001 C CNN
+F 0 "#PWR018" H 5500 7250 50  0001 C CNN
 F 1 "GND" H 5508 7326 50  0000 C CNN
 F 2 "" H 5500 7500 60  0000 C CNN
@@
 	0    1    1    0
 $EndComp
-Wire Wire Line
-	8400 4150 9400 4150
-Connection ~ 9400 4150
 Wire Wire Line
 	8100 4150 7800 4150
@@
 $EndComp
 $Comp
-L GND #PWR14
+L GND #PWR019
 U 1 1 56F62E86
 P 3700 6300
-F 0 "#PWR14" H 3700 6050 50  0001 C CNN
+F 0 "#PWR019" H 3700 6050 50  0001 C CNN
 F 1 "GND" H 3708 6126 50  0000 C CNN
 F 2 "" H 3700 6300 60  0000 C CNN
@@
 $EndComp
 $Comp
-L GND #PWR13
+L GND #PWR020
 U 1 1 56F63D47
 P 3550 7000
-F 0 "#PWR13" H 3550 6750 50  0001 C CNN
+F 0 "#PWR020" H 3550 6750 50  0001 C CNN
 F 1 "GND" H 3558 6826 50  0000 C CNN
 F 2 "" H 3550 7000 60  0000 C CNN
@@
 	3550 7000 3550 6900
 $Comp
-L VAA #PWR12
+L VAA #PWR021
 U 1 1 56F64F84
 P 3550 6000
-F 0 "#PWR12" H 3550 5850 50  0001 C CNN
+F 0 "#PWR021" H 3550 5850 50  0001 C CNN
 F 1 "VAA" H 3570 6174 50  0000 C CNN
 F 2 "" H 3550 6000 60  0000 C CNN
@@
 $EndComp
 $Comp
-L GND #PWR11
+L GND #PWR022
 U 1 1 56F67700
 P 3550 5500
-F 0 "#PWR11" H 3550 5250 50  0001 C CNN
+F 0 "#PWR022" H 3550 5250 50  0001 C CNN
 F 1 "GND" H 3558 5326 50  0000 C CNN
 F 2 "" H 3550 5500 60  0000 C CNN
@@
 	3850 3750 3150 3750
 $Comp
-L +BATT #PWR3
+L +BATT #PWR023
 U 1 1 56F67E62
 P 1400 1500
-F 0 "#PWR3" H 1400 1350 50  0001 C CNN
+F 0 "#PWR023" H 1400 1350 50  0001 C CNN
 F 1 "+BATT" H 1418 1673 50  0000 C CNN
 F 2 "" H 1400 1500 60  0000 C CNN
@@
 Connection ~ 2150 1500
 $Comp
-L +BATT #PWR10
+L +BATT #PWR024
 U 1 1 56F688A0
 P 3550 4900
-F 0 "#PWR10" H 3550 4750 50  0001 C CNN
+F 0 "#PWR024" H 3550 4750 50  0001 C CNN
 F 1 "+BATT" H 3568 5073 50  0000 C CNN
 F 2 "" H 3550 4900 60  0000 C CNN
@@
 	3150 3950 3150 4800
 $Comp
-L GND #PWR8
+L GND #PWR025
 U 1 1 56F6A149
 P 3150 5500
-F 0 "#PWR8" H 3150 5250 50  0001 C CNN
+F 0 "#PWR025" H 3150 5250 50  0001 C CNN
 F 1 "GND" H 3158 5326 50  0000 C CNN
 F 2 "" H 3150 5500 60  0000 C CNN
@@
 	1400 1500 1400 1800
 $Comp
-L GND #PWR4
+L GND #PWR026
 U 1 1 56F68557
 P 1400 2200
-F 0 "#PWR4" H 1400 1950 50  0001 C CNN
+F 0 "#PWR026" H 1400 1950 50  0001 C CNN
 F 1 "GND" H 1408 2026 50  0000 C CNN
 F 2 "" H 1400 2200 60  0000 C CNN
@@
 Connection ~ 11000 4550
 $Comp
-L GND #PWR30
+L GND #PWR027
 U 1 1 570ACE10
 P 11350 4850
-F 0 "#PWR30" H 11350 4600 50  0001 C CNN
+F 0 "#PWR027" H 11350 4600 50  0001 C CNN
 F 1 "GND" H 11358 4676 50  0000 C CNN
 F 2 "" H 11350 4850 60  0000 C CNN
@@
 	8600 2900 8600 2950
 $Comp
-L VCC #PWR21
+L VCC #PWR028
 U 1 1 570ADFB7
 P 7400 1150
-F 0 "#PWR21" H 7400 1000 50  0001 C CNN
+F 0 "#PWR028" H 7400 1000 50  0001 C CNN
 F 1 "VCC" H 7420 1324 50  0000 C CNN
 F 2 "" H 7400 1150 60  0000 C CNN
@@
 $EndComp
 $Comp
-L GND #PWR7
+L GND #PWR029
 U 1 1 570E43C6
 P 2200 1050
-F 0 "#PWR7" H 2200 800 50  0001 C CNN
+F 0 "#PWR029" H 2200 800 50  0001 C CNN
 F 1 "GND" H 2208 876 50  0000 C CNN
 F 2 "" H 2200 1050 60  0000 C CNN
@@
 	3000 1600 3000 950
 $Comp
-L VAA #PWR6
+L VAA #PWR030
 U 1 1 570E46C1
 P 2200 850
-F 0 "#PWR6" H 2200 700 50  0001 C CNN
+F 0 "#PWR030" H 2200 700 50  0001 C CNN
 F 1 "VAA" H 2220 1024 50  0000 C CNN
 F 2 "" H 2200 850 60  0000 C CNN
@@
 Wire Wire Line
 	4150 3150 3150 3150
+Wire Wire Line
+	8400 4150 9050 4150
+Wire Wire Line
+	9050 4150 9050 4950
+Connection ~ 9050 4950
 $EndSCHEMATC
